File: KiCad/high voltage servo drive 3ch/high voltage servo drive 3ch.kicad_sch (KiCad schematic)
At the start: 12 parts

Commit message: prepare rev0.1 for manufacturing
Parts:
- removed H1, H2, H3, H4, H5, H6, H7, H8, H9: MountingHole, footprints:MountingHole_3.2mm_M3, symbol Mechanical:MountingHole
- R147, R149: Generic Allowed? (none) -> yes; LCSC# (none) -> C106231; Manufacturer (none) -> YAGEO; Part number (none) -> RC0402FR-070RL; cost (none) -> 0.0007
- R148: Generic Allowed? (none) -> yes; LCSC# (none) -> C60490; Manufacturer (none) -> YAGEO; Part number (none) -> RC0402FR-0710KL; cost (none) -> 0.0007
