File: KiCad/high voltage servo drive 3ch/communication.kicad_sch (KiCad schematic)
At the start: 75 parts, among them J1 8P8C_LED_Shielded_x2, M1 Fan_4pin, U10 TPS54202DDC, U3 MAX13433EESD, U4 MAX13433EESD, U5 CA_IS3741HW, U6 R24C2T25-R, U7 CA_IS3741HW, U8 CA_IS3741HW, U9 74LVC1G126

Commit message: prepare rev0.1 for manufacturing
Parts:
- removed C24: 330pf, Capacitor_SMD:C_0402_1005Metric, symbol Device:C
- removed C39: .1uf, Capacitor_SMD:C_0402_1005Metric, symbol Device:C
- removed C41: 2.2uf, Capacitor_SMD:C_1206_3216Metric, symbol Device:C
- removed D11: GATE_SUPPLY_ON, LED_SMD:LED_0603_1608Metric, symbol Device:LED
- removed R16: 68.1k, Resistor_SMD:R_0402_1005Metric, symbol Device:R_US
- removed R31: 10k, Resistor_SMD:R_0402_1005Metric, symbol Device:R_US
- removed TP1: GATE_SUPPLY, TestPoint:TestPoint_Pad_D2.0mm, symbol Connector:TestPoint
- removed U6: R24C2T25-R, footprints:36L-SSOP_RCP, symbol R24C2T25-R:R24C2T25-R
- added D54: LED, LED_SMD:LED_0603_1608Metric, symbol Device:LED
- added PS1: F0505S-1W, footprints:Converter_DCDC_FXXS-1W, symbol F0505S-1W:F0505S-1W
- added R153, R154, R155, R156: 0, Resistor_SMD:R_0402_1005Metric, symbol Device:R_US
- added TP3: 5V, TestPoint:TestPoint_Pad_D2.0mm, symbol Connector:TestPoint
- C138, C22, C23, C25, C26, C31, C32, C33, C37, C42, C43, C44: Generic Allowed? (none) -> yes; LCSC# (none) -> C105882; Manufacturer (none) -> YAGEO; Part number (none) -> CC0402KRX5R9BB104; cost (none) -> 0.003
- C27, C34, C35: Generic Allowed? (none) -> yes; LCSC# C473196 -> C7471876; Manufacturer (none) -> KNSCHA; Part number (none) -> 189RV0014; cost (none) -> 0.05
- C28, C29: Generic Allowed? (none) -> yes; LCSC# (none) -> C12891; Manufacturer (none) -> Samsung Electro-Mechanics; Part number (none) -> CL31A226KAHNNNE; cost (none) -> 0.04
- C30: Generic Allowed? (none) -> yes; LCSC# (none) -> C107010; Manufacturer (none) -> YAGEO; Part number (none) -> CC0402JRNPO9BN750; cost (none) -> 0.0011
- C36, C38: Generic Allowed? (none) -> yes; LCSC# C7393943 -> C50254; Manufacturer (none) -> Samsung Electro-Mechanics; Part number (none) -> CL31B225KBHNNNE; cost (none) -> 0.03
- C40: value .1uf -> 22uf; footprint Capacitor_SMD:C_0402_1005Metric -> Capacitor_SMD:C_1206_3216Metric; Generic Allowed? (none) -> yes; LCSC# (none) -> C12891; Manufacturer (none) -> Samsung Electro-Mechanics; Part number (none) -> CL31A226KAHNNNE; cost (none) -> 0.04
- C52, M1, TP10, TP11, TP12, TP13, TP14, TP2, TP5, TP8, TP9: now not fitted
- D10: value 24V_ISO_ON -> LED; Generic Allowed? (none) -> yes; LCSC# (none) -> C965807; Manufacturer (none) -> XINGLIGHT; Part number (none) -> XL-1608UBC-04; cost (none) -> 0.004
- D5, D6, D7, D8: LCSC# (none) -> C5199207; Manufacturer SMC Diode Solutions -> ElecSuper; Part number SM712 -> CDSOT23-SM712-ES; cost (none) -> 0.03
- D9: value 5V_ISO_ON -> LED; Generic Allowed? (none) -> yes; LCSC# (none) -> C965807; Manufacturer (none) -> XINGLIGHT; Part number (none) -> XL-1608UBC-04; cost (none) -> 0.004
- FB1, FB2: value FerriteBead -> 0; Generic Allowed? (none) -> yes; LCSC# C963878 -> C2907406; Manufacturer (none) -> FOJAN; Part number (none) -> FRC1206P000 TS; cost (none) -> 0.0015
- J1: Generic Allowed? (none) -> yes; Manufacturer (none) -> Lian Xin Technology; Part number (none) -> XDRJ-1609-002; cost (none) -> 1.08; now not fitted
- L1: Generic Allowed? (none) -> yes; Manufacturer (none) -> CND-tek; Part number (none) -> CND-WCM0805M801-2; cost (none) -> 0.02
- L2, L3, L4: Generic Allowed? (none) -> yes; LCSC# C193073 -> C3020807; Manufacturer (none) -> CND-tek; Part number (none) -> CND-WCM0805M801-2; cost (none) -> 0.02
- L5: footprint Inductor_SMD:L_Taiyo-Yuden_MD-4040 -> footprints:CY54_INDUCTOR; Generic Allowed? (none) -> yes; LCSC# (none) -> C2929432; Manufacturer (none) -> SHOU HAN; Part number (none) -> CY54-15UH; cost (none) -> 0.05
- R146, R30: Generic Allowed? (none) -> yes; LCSC# (none) -> C60490; Manufacturer (none) -> YAGEO; Part number (none) -> RC0402FR-0710KL; cost (none) -> 0.0007
- R15: value 11k -> 1k; Generic Allowed? (none) -> yes, 1% or better; LCSC# (none) -> C106235; Manufacturer (none) -> YAGEO; Part number (none) -> RC0402FR-071KL; cost (none) -> 0.0007
- R17, R18, R19, R20, R29: Generic Allowed? (none) -> yes, 1% or better; LCSC# (none) -> C106235; Manufacturer (none) -> YAGEO; Part number (none) -> RC0402FR-071KL; cost (none) -> 0.0007
- R21: Generic Allowed? (none) -> yes; LCSC# (none) -> C60491; Manufacturer (none) -> YAGEO; Part number (none) -> RC0402FR-07100KL; cost (none) -> 0.0007
- R22: Generic Allowed? (none) -> yes; LCSC# (none) -> C274352; Manufacturer (none) -> YAGEO; Part number (none) -> RC0402FR-0713K3L; cost (none) -> 0.0007
- R23: value 500k -> 560k; Generic Allowed? (none) -> yes; LCSC# (none) -> C137958; Manufacturer (none) -> YAGEO; Part number (none) -> RC0402FR-07560KL; cost (none) -> 0.0007; now not fitted
- R24: Generic Allowed? (none) -> yes; LCSC# (none) -> C60491; Manufacturer (none) -> YAGEO; Part number (none) -> RC0402FR-07100KL; cost (none) -> 0.0007; now not fitted
- R97, R98: Generic Allowed? (none) -> yes; LCSC# (none) -> C114758; Manufacturer (none) -> YAGEO; Part number (none) -> RC0402FR-07120RL; cost (none) -> 0.0008
- U10: Manufacturer (none) -> TI; Part number (none) -> TPS54202DDCR; cost (none) -> 0.10
- U5, U7, U8: Manufacturer (none) -> Chipanalog; Part number (none) -> CA-IS3741HW; cost (none) -> 0.70
- U9: Manufacturer (none) -> GR; Part number (none) -> 74LVC1G126CT05ARCQ; cost (none) -> 0.03
Connections:
- net +24V: now also R154.2, R155.2; no longer C35.1, C38.2, C40.2, M1.2 (+)
- net +5V: now also R153.2, R156.2
- net GND: now also PS1.2 (-Vin); no longer C40.1
- net GND1: now also C40.1, D54.1 (K), PS1.5 (-Vout); no longer R15.1
- net +5VP: now reaches R15.2
- net +5VP: now also C40.2, PS1.7 (+Vout), TP3.1
- new net: C35.1, M1.2 (+), R155.1, R156.1
- new net: D54.2 (A), R15.1
- new net: C38.2, PS1.1 (+Vin), R153.1, R154.1
Other:
- note removed: "GATE_SUPPLY voltage must be set according to which IPMs are used IGBT: 15v SiC: 18v"
- note removed: "Voltage adjust 15v: 54.9k 18v: 68.1k"
- moved on the sheet: C35

Commit message: update BOM and change transceivers
Parts:
- removed U3, U4: MAX13433EESD, Package_SO:SOIC-14_3.9x8.7mm_P1.27mm, symbol Interface_UART:MAX13433EESD
- added U3, U4: SP491EEN-L/TR, Package_SO:SOIC-14_3.9x8.7mm_P1.27mm, symbol THVD1452:THVD1452
- FB1, FB2: LCSC# C2907406 -> C2907288; Part number FRC1206P000 TS -> FRC0805P000 TS
- J1: now fitted
- U10, U5, U7, U8: Generic Allowed? (none) -> no
- U9: Generic Allowed? (none) -> yes
Connections:
- net +5V: now also U3.13 (VCC), U3.14 (VCC), U3.4 (DE), U4.13 (VCC), U4.14 (VCC)
- net GND: now also U3.3 (~{RE}), U3.6 (GND), U3.7 (NC), U4.6 (GND), U4.7 (NC)
- net RX_ISO: now also U3.2 (RO), U4.5 (DI)
- net RX_PASSTHROUGH_ENABLE_ISO: now also U4.4 (DE)
- net TX_PASSTHROUGH_DISABLE_ISO: now also U4.3 (~{RE})
- net TX_SNOOP_ISO: now also U3.5 (DI), U4.2 (RO)
- net at L4.2: now also U4.10 (~{Z})
- net at L3.2, R98.2: now also U4.11 (~{B})
- net at L3.4, R98.1: now also U4.12 (A)
- net at L4.4: now also U4.9 (Y)
- net at L2.2: now also U3.10 (~{Z})
- net at L2.4: now also U3.9 (Y)
- net at L1.4, R97.1: now also U3.12 (A)
- net at L1.2, R97.2: now also U3.11 (~{B})
Other:
- note added: "THVD1452 is pin compatible with SP491EEN-L/TR THVD1452: 50 Mbit SP491EEN-L/TR: 10Mbit"
