File: KiCad/high voltage servo drive 3ch/communication.kicad_sch (KiCad schematic)
At the start: 74 parts, among them J1 8P8C_LED_Shielded_x2, M1 Fan_4pin, U10 TPS54202DDC, U3 SP491EEN-L/TR, U4 SP491EEN-L/TR, U5 CA_IS3741HW, U7 CA_IS3741HW, U8 CA_IS3741HW, U9 74LVC1G126

Commit message: add rev 0.2 changes and rev 0.1 mfg files
Parts:
- D10, D54, D9: LCSC# C965807 -> C965804; Part number XL-1608UBC-04 -> XL-1608UGC-04; cost 0.004 -> 0.005
- J1, PS1: now not fitted
- R22: Generic Allowed? yes -> yes, 1% or better
Changed lines of the file:
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@@
 			)
 		)
-		(property "Description" "Light emitting diode"
+		(property "Description" "LED, emerald green"
 			(at 473.71 302.26 0)
 			(effects
@@
 			)
 		)
-		(property "cost" "0.004"
+		(property "cost" "0.005"
 			(at 473.71 302.26 0)
 			(effects
@@
 			)
 		)
-		(property "LCSC#" "C965807"
+		(property "LCSC#" "C965804"
 			(at 473.71 302.26 0)
 			(effects
@@
 			)
 		)
-		(property "Part number" "XL-1608UBC-04"
+		(property "Part number" "XL-1608UGC-04"
 			(at 473.71 302.26 0)
 			(effects
@@
 			)
 		)
-		(property "Generic Allowed?" "yes"
+		(property "Generic Allowed?" "yes, 1% or better"
 			(at 278.13 299.72 0)
 			(effects
@@
 			)
 		)
-		(property "Description" "Light emitting diode"
+		(property "Description" "LED, emerald green"
 			(at 314.96 292.1 0)
 			(effects
@@
 			)
 		)
-		(property "cost" "0.004"
+		(property "cost" "0.005"
 			(at 314.96 292.1 0)
 			(effects
@@
 			)
 		)
-		(property "LCSC#" "C965807"
+		(property "LCSC#" "C965804"
 			(at 314.96 292.1 0)
 			(effects
@@
 			)
 		)
-		(property "Part number" "XL-1608UBC-04"
+		(property "Part number" "XL-1608UGC-04"
 			(at 314.96 292.1 0)
 			(effects
@@
 		(in_bom yes)
 		(on_board yes)
-		(dnp no)
+		(dnp yes)
 		(fields_autoplaced yes)
 		(property "Reference" "J1"
@@
 			)
 		)
-		(property "Description" "Light emitting diode"
+		(property "Description" "LED, emerald green"
 			(at 158.75 292.1 0)
 			(effects
@@
 			)
 		)
-		(property "cost" "0.004"
+		(property "cost" "0.005"
 			(at 158.75 292.1 0)
 			(effects
@@
 			)
 		)
-		(property "LCSC#" "C965807"
+		(property "LCSC#" "C965804"
 			(at 158.75 292.1 0)
 			(effects
@@
 			)
 		)
-		(property "Part number" "XL-1608UBC-04"
+		(property "Part number" "XL-1608UGC-04"
 			(at 158.75 292.1 0)
 			(effects
@@
 		(in_bom yes)
 		(on_board yes)
-		(dnp no)
+		(dnp yes)
 		(fields_autoplaced yes)
 		(property "Reference" "PS1"
@@
 		(in_bom yes)
 		(on_board yes)
-		(dnp no)
+		(dnp yes)
 		(fields_autoplaced yes)
 		(property "Reference" "J1"

Commit message: update bom
Parts:
- C52: Generic Allowed? (none) -> yes
Changed lines of the file:
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@@
 	)
 	(symbol
-		(lib_name "THVD1452:THVD1452")
 		(lib_id "THVD1452:THVD1452")
 		(at 294.64 124.46 0)
@@
 			)
 		)
+		(property "Generic Allowed?" "yes"
+			(at 373.38 342.9 0)
+			(effects
+				(font
+					(size 1.27 1.27)
+				)
+				(hide yes)
+			)
+		)
 		(pin "1"
 		)
@@
 	)
 	(symbol
-		(lib_name "THVD1452:THVD1452")
 		(lib_id "THVD1452:THVD1452")
 		(at 294.64 176.53 0)
