File: KiCad/high voltage servo drive 3ch/current_sense.kicad_sch (KiCad schematic)
At the start: 126 parts, among them U12 OPA4323IPWR, U13 OPA4323IPWR, U14 OPA4323IPWR

Commit message: prepare rev0.1 for manufacturing
Parts:
- C100, C103, C105, C106, C54, C55, C58, C59, C62, C63, C66, C68, C69, C72, C74, C75, C78, C80, C81, C84, C86, C87, C91, C93, C94, C97, C99: Generic Allowed? (none) -> yes; LCSC# (none) -> C282238; Manufacturer (none) -> YAGEO; Part number (none) -> CC0402BRNPO9BN1R5
- C101, C107, C109, C56, C57, C64, C70, C76, C82, C88, C90, C95: value 0.1uf -> .1uf; Generic Allowed? (none) -> yes; LCSC# (none) -> C105882; Manufacturer (none) -> YAGEO; Part number (none) -> CC0402KRX5R9BB104; cost (none) -> 0.003
- C102, C108, C60, C65, C71, C77, C83, C89, C96: Generic Allowed? (none) -> yes; LCSC# (none) -> C106200; Manufacturer (none) -> YAGEO; Part number (none) -> CC0402JRNPO9BN101; cost (none) -> 0.0011
- C201, C202, C203: Generic Allowed? (none) -> yes; LCSC# (none) -> C14445; Manufacturer (none) -> Samsung Electro-Mechanics; Part number (none) -> CL05A105KP5NNNC; cost (none) -> 0.0017
- D13, D14, D15, D16, D17, D18, D19, D20, D21, D22, D23, D24, D25, D26, D27, D28, D29, D30: LCSC# (none) -> C12765; Manufacturer onsemi -> LRC; Part number BAT54SLT1G -> LBAT54SLT1G; cost (none) -> 0.01
- R33, R34, R38, R39, R43, R44, R48, R49, R53, R54, R58, R59, R63, R64, R68, R69, R73, R74: value 1k -> 1k; Generic Allowed? (none) -> yes, 1% or better; LCSC# (none) -> C106235; Manufacturer (none) -> YAGEO; Part number (none) -> RC0402FR-071KL; cost (none) -> 0.0007
- R35, R36, R40, R41, R45, R46, R50, R51, R55, R56, R60, R61, R65, R66, R70, R71, R75, R76: value 12.1 -> 12.1k; Generic Allowed? (none) -> yes, 1% or better; LCSC# (none) -> C132157; Manufacturer (none) -> YAGEO; Part number (none) -> RC0402FR-0712K1L; cost (none) -> 0.0007
- R37, R42, R47, R52, R57, R62, R67, R72, R77: Generic Allowed? (none) -> yes; LCSC# (none) -> C477760; Manufacturer (none) -> YAGEO; Part number (none) -> RC0402JR-0750RL; cost (none) -> 0.0007
- U12, U13, U14: Manufacturer (none) -> TI; Part number (none) -> OPA4323IPWR; cost (none) -> 0.87

Commit message: update BOM and change transceivers
Parts:
- U12, U13, U14: Generic Allowed? (none) -> no
