File: KiCad/high voltage servo drive 3ch/current_sense.kicad_sch (KiCad schematic)
At the start: 126 parts, among them U12 OPA4323IPWR, U13 OPA4323IPWR, U14 OPA4323IPWR

Commit message: add rev 0.2 changes and rev 0.1 mfg files
Connections:
- net at C100.1, C97.2, C98.1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: now also U14.6 (-); no longer U14.5 (+)
- net at C104.2, C105.1, D29.3 (common)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: now also U14.10 (+); no longer U14.9 (-)
- net at C85.2, C86.1, D23.3 (common)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: now also U13.10 (+); no longer U13.9 (-)
- net at C53.1, C55.2, C59.1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: now also U12.2 (-); no longer U12.3 (+)
- net at C73.2, C74.1, D19.3 (common)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: now also U13.3 (+); no longer U13.2 (-)
- net at C72.2, C73.1, C75.1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: now also U13.2 (-); no longer U13.3 (+)
- net at C84.2, C85.1, C87.1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: now also U13.9 (-); no longer U13.10 (+)
- net at C53.2, C54.1, D13.3 (common)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: now also U12.3 (+); no longer U12.2 (-)
- net at C103.2, C104.1, C106.1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: now also U14.9 (-); no longer U14.10 (+)
- net at C78.2, C79.1, C81.1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: now also U13.6 (-); no longer U13.5 (+)
- net at C91.2, C92.1, C94.1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: now also U14.2 (-); no longer U14.3 (+)
- net at C58.2, C61.1, C63.1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: now also U12.6 (-); no longer U12.5 (+)
- net at C61.2, C62.1, D15.3 (common)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: now also U12.5 (+); no longer U12.6 (-)
- net at C92.2, C93.1, D25.3 (common)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: now also U14.3 (+); no longer U14.2 (-)
- net at C79.2, C80.1, D21.3 (common)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: now also U13.5 (+); no longer U13.6 (-)
- net at C66.2, C67.1, C69.1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: now also U12.9 (-); no longer U12.10 (+)
- net at C67.2, C68.1, D17.3 (common)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: now also U12.10 (+); no longer U12.9 (-)
- net at C98.2, C99.1, D27.3 (common)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: now also U14.5 (+); no longer U14.6 (-)
Changed lines of the file:
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@@
 		(lib_id "Amplifier_Operational:OPA4340UA")
 		(at 130.81 60.96 0)
+		(mirror x)
 		(unit 1)
 		(exclude_from_sim no)
@@
 		(on_board yes)
 		(dnp no)
-		(fields_autoplaced yes)
 		(property "Reference" "U12"
-			(at 130.81 50.8 0)
+			(at 130.81 71.12 0)
 			(effects
 				(font
@@
 		)
 		(property "Value" "OPA4323IPWR"
-			(at 130.81 53.34 0)
+			(at 130.81 68.58 0)
 			(effects
 				(font
@@
 		)
 		(property "Footprint" "Package_SO:TSSOP-14_4.4x5mm_P0.65mm"
-			(at 129.54 58.42 0)
+			(at 129.54 63.5 0)
 			(effects
 				(font
@@
 		)
 		(property "Datasheet" "http://www.ti.com/lit/ds/symlink/opa340.pdf"
-			(at 132.08 55.88 0)
+			(at 132.08 66.04 0)
 			(effects
 				(font
@@
 		(lib_id "Amplifier_Operational:OPA4340UA")
 		(at 508 285.75 0)
+		(mirror x)
 		(unit 3)
 		(exclude_from_sim no)
@@
 		(on_board yes)
 		(dnp no)
-		(fields_autoplaced yes)
 		(property "Reference" "U14"
-			(at 508 275.59 0)
+			(at 508 295.91 0)
 			(effects
 				(font
@@
 		)
 		(property "Value" "OPA4323IPWR"
-			(at 508 278.13 0)
+			(at 508 293.37 0)
 			(effects
 				(font
@@
 		)
 		(property "Footprint" "Package_SO:TSSOP-14_4.4x5mm_P0.65mm"
-			(at 506.73 283.21 0)
+			(at 506.73 288.29 0)
 			(effects
 				(font
@@
 		)
 		(property "Datasheet" "http://www.ti.com/lit/ds/symlink/opa340.pdf"
-			(at 509.27 280.67 0)
+			(at 509.27 290.83 0)
 			(effects
 				(font
@@
 		(lib_id "Amplifier_Operational:OPA4340UA")
 		(at 317.5 62.23 0)
+		(mirror x)
 		(unit 2)
 		(exclude_from_sim no)
@@
 		(on_board yes)
 		(dnp no)
-		(fields_autoplaced yes)
 		(property "Reference" "U12"
-			(at 317.5 52.07 0)
+			(at 317.5 72.39 0)
 			(effects
 				(font
@@
 		)
 		(property "Value" "OPA4323IPWR"
-			(at 317.5 54.61 0)
+			(at 317.5 69.85 0)
 			(effects
 				(font
@@
 		)
 		(property "Footprint" "Package_SO:TSSOP-14_4.4x5mm_P0.65mm"
-			(at 316.23 59.69 0)
+			(at 316.23 64.77 0)
 			(effects
 				(font
@@
 		)
 		(property "Datasheet" "http://www.ti.com/lit/ds/symlink/opa340.pdf"
-			(at 318.77 57.15 0)
+			(at 318.77 67.31 0)
 			(effects
 				(font
@@
 		(lib_id "Amplifier_Operational:OPA4340UA")
 		(at 508 172.72 0)
+		(mirror x)
 		(unit 3)
 		(exclude_from_sim no)
@@
 		(on_board yes)
 		(dnp no)
-		(fields_autoplaced yes)
 		(property "Reference" "U13"
-			(at 508 162.56 0)
+			(at 508 182.88 0)
 			(effects
 				(font
@@
 		)
 		(property "Value" "OPA4323IPWR"
-			(at 508 165.1 0)
+			(at 508 180.34 0)
 			(effects
 				(font
@@
 		)
 		(property "Footprint" "Package_SO:TSSOP-14_4.4x5mm_P0.65mm"
-			(at 506.73 170.18 0)
+			(at 506.73 175.26 0)
 			(effects
 				(font
@@
 		)
 		(property "Datasheet" "http://www.ti.com/lit/ds/symlink/opa340.pdf"
-			(at 509.27 167.64 0)
+			(at 509.27 177.8 0)
 			(effects
 				(font
@@
 		(lib_id "Amplifier_Operational:OPA4340UA")
 		(at 130.81 285.75 0)
+		(mirror x)
 		(unit 1)
 		(exclude_from_sim no)
@@
 		(on_board yes)
 		(dnp no)
-		(fields_autoplaced yes)
 		(property "Reference" "U14"
-			(at 130.81 275.59 0)
+			(at 130.81 295.91 0)
 			(effects
 				(font
@@
 		)
 		(property "Value" "OPA4323IPWR"
-			(at 130.81 278.13 0)
+			(at 130.81 293.37 0)
 			(effects
 				(font
@@
 		)
 		(property "Footprint" "Package_SO:TSSOP-14_4.4x5mm_P0.65mm"
-			(at 129.54 283.21 0)
+			(at 129.54 288.29 0)
 			(effects
 				(font
@@
 		)
 		(property "Datasheet" "http://www.ti.com/lit/ds/symlink/opa340.pdf"
-			(at 132.08 280.67 0)
+			(at 132.08 290.83 0)
 			(effects
 				(font
@@
 		(lib_id "Amplifier_Operational:OPA4340UA")
 		(at 508 60.96 0)
+		(mirror x)
 		(unit 3)
 		(exclude_from_sim no)
@@
 		(on_board yes)
 		(dnp no)
-		(fields_autoplaced yes)
 		(property "Reference" "U12"
-			(at 508 50.8 0)
+			(at 508 71.12 0)
 			(effects
 				(font
@@
 		)
 		(property "Value" "OPA4323IPWR"
-			(at 508 53.34 0)
+			(at 508 68.58 0)
 			(effects
 				(font
@@
 		)
 		(property "Footprint" "Package_SO:TSSOP-14_4.4x5mm_P0.65mm"
-			(at 506.73 58.42 0)
+			(at 506.73 63.5 0)
 			(effects
 				(font
@@
 		)
 		(property "Datasheet" "http://www.ti.com/lit/ds/symlink/opa340.pdf"
-			(at 509.27 55.88 0)
+			(at 509.27 66.04 0)
 			(effects
 				(font
@@
 		(lib_id "Amplifier_Operational:OPA4340UA")
 		(at 317.5 173.99 0)
+		(mirror x)
 		(unit 2)
 		(exclude_from_sim no)
@@
 		(on_board yes)
 		(dnp no)
-		(fields_autoplaced yes)
 		(property "Reference" "U13"
-			(at 317.5 163.83 0)
+			(at 317.5 184.15 0)
 			(effects
 				(font
@@
 		)
 		(property "Value" "OPA4323IPWR"
-			(at 317.5 166.37 0)
+			(at 317.5 181.61 0)
 			(effects
 				(font
@@
 		)
 		(property "Footprint" "Package_SO:TSSOP-14_4.4x5mm_P0.65mm"
-			(at 316.23 171.45 0)
+			(at 316.23 176.53 0)
 			(effects
 				(font
@@
 		)
 		(property "Datasheet" "http://www.ti.com/lit/ds/symlink/opa340.pdf"
-			(at 318.77 168.91 0)
+			(at 318.77 179.07 0)
 			(effects
 				(font
@@
 		(lib_id "Amplifier_Operational:OPA4340UA")
 		(at 317.5 287.02 0)
+		(mirror x)
 		(unit 2)
 		(exclude_from_sim no)
@@
 		(on_board yes)
 		(dnp no)
-		(fields_autoplaced yes)
 		(property "Reference" "U14"
-			(at 317.5 276.86 0)
+			(at 317.5 297.18 0)
 			(effects
 				(font
@@
 		)
 		(property "Value" "OPA4323IPWR"
-			(at 317.5 279.4 0)
+			(at 317.5 294.64 0)
 			(effects
 				(font
@@
 		)
 		(property "Footprint" "Package_SO:TSSOP-14_4.4x5mm_P0.65mm"
-			(at 316.23 284.48 0)
+			(at 316.23 289.56 0)
 			(effects
 				(font
@@
 		)
 		(property "Datasheet" "http://www.ti.com/lit/ds/symlink/opa340.pdf"
-			(at 318.77 281.94 0)
+			(at 318.77 292.1 0)
 			(effects
 				(font
@@
 		(lib_id "Amplifier_Operational:OPA4340UA")
 		(at 130.81 172.72 0)
+		(mirror x)
 		(unit 1)
 		(exclude_from_sim no)
@@
 		(on_board yes)
 		(dnp no)
-		(fields_autoplaced yes)
 		(property "Reference" "U13"
-			(at 130.81 162.56 0)
+			(at 130.81 182.88 0)
 			(effects
 				(font
@@
 		)
 		(property "Value" "OPA4323IPWR"
-			(at 130.81 165.1 0)
+			(at 130.81 180.34 0)
 			(effects
 				(font
@@
 		)
 		(property "Footprint" "Package_SO:TSSOP-14_4.4x5mm_P0.65mm"
-			(at 129.54 170.18 0)
+			(at 129.54 175.26 0)
 			(effects
 				(font
@@
 		)
 		(property "Datasheet" "http://www.ti.com/lit/ds/symlink/opa340.pdf"
-			(at 132.08 167.64 0)
+			(at 132.08 177.8 0)
 			(effects
 				(font

Commit message: update bom
Parts:
- C104, C53, C61, C67, C73, C79, C85, C92, C98: Generic Allowed? (none) -> yes
Changed lines of the file:
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@@
 			)
 		)
+		(property "Generic Allowed?" "yes"
+			(at 101.6 172.72 0)
+			(effects
+				(font
+					(size 1.27 1.27)
+				)
+				(hide yes)
+			)
+		)
 		(pin "2"
 		)
@@
 			)
 		)
+		(property "Generic Allowed?" "yes"
+			(at 478.79 60.96 0)
+			(effects
+				(font
+					(size 1.27 1.27)
+				)
+				(hide yes)
+			)
+		)
 		(pin "2"
 		)
@@
 			)
 		)
+		(property "Generic Allowed?" "yes"
+			(at 101.6 60.96 0)
+			(effects
+				(font
+					(size 1.27 1.27)
+				)
+				(hide yes)
+			)
+		)
 		(pin "2"
 		)
@@
 			)
 		)
+		(property "Generic Allowed?" "yes"
+			(at 101.6 285.75 0)
+			(effects
+				(font
+					(size 1.27 1.27)
+				)
+				(hide yes)
+			)
+		)
 		(pin "2"
 		)
@@
 			)
 		)
+		(property "Generic Allowed?" "yes"
+			(at 478.79 172.72 0)
+			(effects
+				(font
+					(size 1.27 1.27)
+				)
+				(hide yes)
+			)
+		)
 		(pin "2"
 		)
@@
 			)
 		)
+		(property "Generic Allowed?" "yes"
+			(at 288.29 62.23 0)
+			(effects
+				(font
+					(size 1.27 1.27)
+				)
+				(hide yes)
+			)
+		)
 		(pin "2"
 		)
@@
 			)
 		)
+		(property "Generic Allowed?" "yes"
+			(at 478.79 285.75 0)
+			(effects
+				(font
+					(size 1.27 1.27)
+				)
+				(hide yes)
+			)
+		)
 		(pin "2"
 		)
@@
 			)
 		)
+		(property "Generic Allowed?" "yes"
+			(at 288.29 173.99 0)
+			(effects
+				(font
+					(size 1.27 1.27)
+				)
+				(hide yes)
+			)
+		)
 		(pin "2"
 		)
@@
 			(at 288.29 287.02 0)
 			(effects
+				(font
+					(size 1.27 1.27)
+				)
+				(hide yes)
+			)
+		)
+		(property "Generic Allowed?" "yes"
+			(at 288.29 287.02 0)
+			(effects
