File: KiCad/high voltage servo drive 3ch/high voltage servo drive 3ch.kicad_pcb (KiCad board)
At the start: 4 copper layers, 109 x 231.4 mm, 486 parts, among them J1 8P8C_LED_Shielded_x2, J3 Conn_ARM_SWD_TagConnect_TC2030, J4 MOTOR_A, J5 MOTOR_B, J6 MOTOR_C, J7 DC BUS, J8 STO, M1 Fan_4pin, Q1 BSS83P, U1 STM32G473QET6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

Commit message: update BOM and change transceivers
Parts:
- U15, U16, U19: footprint Package_DIP:DIP-4_W7.62mm_SMDSocket_SmallPads -> Package_DIP:DIP-4_W7.62mm
- U20: footprint Package_SO:PowerIntegrations_SO-8C -> Package_SO:PowerIntegrations_SO-8B
- U3, U4: value MAX13433EESD -> THVD1452
- moved U19 4.02 mm to (262.9, 206.1)
- moved U15 4.00 mm to (248.4, 213.7)
- moved U16 4.00 mm to (254.4, 213.7)
Connections:
- U3 pad 1: +5V -> (no net)
- U3 pad 13: unconnected-(U3-NC-Pad13) -> +5V
- U3 pad 3: +5V -> GND
- U3 pad 4: GND -> +5V
- U3 pad 7: unconnected-(U3-NC-Pad7) -> GND
- U3 pad 8: GND -> (no net)
- U4 pad 1: +5V -> (no net)
- U4 pad 13: unconnected-(U4-NC-Pad13) -> +5V
- U4 pad 3: /Communication/RX_PASSTHROUGH_ENABLE_ISO -> /Communication/TX_PASSTHROUGH_DISABLE_ISO
- U4 pad 4: /Communication/TX_PASSTHROUGH_DISABLE_ISO -> /Communication/RX_PASSTHROUGH_ENABLE_ISO
- U4 pad 7: unconnected-(U4-NC-Pad7) -> GND
- U4 pad 8: GND -> (no net)
Routing:
- net +5V: track 41.4 -> 35.0 mm, vias 16 -> 17
- net /Communication/RX_PASSTHROUGH_ENABLE_ISO: track 14.2 -> 18.5 mm
- net /Communication/TX_PASSTHROUGH_DISABLE_ISO: track 20.9 -> 19.8 mm
- net GND: track 49.8 -> 50.2 mm, vias 30 -> 28
Other:
- board text added: "commit: f7b9e71"
- board text added: "github.com/ExcessiveOverkill/hvsd-3ch"
- board text removed: "####"
