File: KiCad/high voltage servo drive 3ch/high voltage servo drive 3ch.kicad_pcb (KiCad board)
At the start: 4 copper layers, 109 x 231.4 mm, 487 parts, among them J1 8P8C_LED_Shielded_x2, J3 Conn_ARM_SWD_TagConnect_TC2030, J4 MOTOR_A, J5 MOTOR_B, J6 MOTOR_C, J7 DC BUS, J8 STO, M1 Fan_4pin, Q1 BSS83P, U1 STM32G473QET6, U10 TPS54202DDC, U12 OPA4323IPWR, U13 OPA4323IPWR, U14 OPA4323IPWR, U15 PC-817S1-CTP1-F, U16 PC-817S1-CTP1-F, U17 IPM, U18 IPM, U19 PC-817S1-CTP1-F, U2 IPM, U20 LNK306D, U21 TLV75733PDBV, U3 SP491EEN-L/TR, U4 SP491EEN-L/TR, U5 CA_IS3741HW, U6 TLV75733PDBV, U7 CA_IS3741HW, U8 CA_IS3741HW, U9 74LVC1G126, X1 25Mhz

Commit message: update manufacturing files for rev 0.2
Other:
- board text added: "commit: 9db8997"
- board text removed: "commit:"
Changed lines of the file:
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@@
 		)
 	)
-	(gr_text "commit: "
+	(gr_text "commit: 9db8997"
 		(at 163.6 192.95 0)
 		(layer "F.SilkS")
