File: KiCad/high voltage servo drive 3ch/microcontroller.kicad_sch (KiCad schematic)
At the start: 73 parts, among them J3 Conn_ARM_SWD_TagConnect_TC2030, U1 STM32G473QET6, U11 TPS54202DDC, X1 SG-8002CE

Commit message: prepare rev0.1 for manufacturing
Parts:
- removed C137: 2.2uf, Capacitor_SMD:C_1206_3216Metric, symbol Device:C
- removed C45: 22uf, Capacitor_SMD:CP_Elec_6.3x5.9, symbol Device:C_Polarized
- removed C46, C47: .1uf, Capacitor_SMD:C_0402_1005Metric, symbol Device:C
- removed C48: 75pf, Capacitor_SMD:C_0402_1005Metric, symbol Device:C
- removed C49, C50, C51: 22uf, Capacitor_SMD:C_1206_3216Metric, symbol Device:C
- removed FB3, FB4: FerriteBead, Inductor_SMD:L_0805_2012Metric, symbol Device:FerriteBead
- removed L6: 15uH, Inductor_SMD:L_Taiyo-Yuden_MD-4040, symbol Device:L
- removed R25: 500k, Resistor_SMD:R_0402_1005Metric, symbol Device:R_US
- removed R26, R27: 100k, Resistor_SMD:R_0402_1005Metric, symbol Device:R_US
- removed R28: 13.3k, Resistor_SMD:R_0402_1005Metric, symbol Device:R_US
- removed U11: TPS54202DDC, Package_TO_SOT_SMD:SOT-23-6, symbol Regulator_Switching:TPS54202DDC
- added C24, C39, C41: 22uf, Capacitor_SMD:C_1206_3216Metric, symbol Device:C
- added R151: 120, Resistor_SMD:R_0402_1005Metric, symbol Device:R_US
- added U21, U6: TLV75733PDBV, Package_TO_SOT_SMD:SOT-23-5, symbol Regulator_Linear:TLV75733PDBV
- C110, C111: Generic Allowed? (none) -> yes; LCSC# (none) -> C12891; Manufacturer (none) -> Samsung Electro-Mechanics; Part number (none) -> CL31A226KAHNNNE; cost (none) -> 0.04
- C112, C113, C114, C115, C116, C117, C118, C119, C121, C122, C124, C125, C191, C192, C193, C198, C199, C200: Generic Allowed? (none) -> yes; LCSC# (none) -> C105882; Manufacturer (none) -> YAGEO; Part number (none) -> CC0402KRX5R9BB104; cost (none) -> 0.003
- C120, C123: Generic Allowed? (none) -> yes; LCSC# (none) -> C14445; Manufacturer (none) -> Samsung Electro-Mechanics; Part number (none) -> CL05A105KP5NNNC; cost (none) -> 0.0017
- C126: Generic Allowed? (none) -> yes; LCSC# (none) -> C106200; Manufacturer (none) -> YAGEO; Part number (none) -> CC0402JRNPO9BN101; cost (none) -> 0.0011
- C127: value 75pf -> 100pf; Generic Allowed? (none) -> yes; LCSC# (none) -> C106200; Manufacturer (none) -> YAGEO; Part number (none) -> CC0402JRNPO9BN101; cost (none) -> 0.0011
- C194: Generic Allowed? (none) -> yes; LCSC# C7393943 -> C50254; Manufacturer (none) -> Samsung Electro-Mechanics; Part number (none) -> CL31B225KBHNNNE; cost (none) -> 0.03
- D12: value 3.3V_ON -> LED; Generic Allowed? (none) -> yes; LCSC# (none) -> C965807; Manufacturer (none) -> XINGLIGHT; Part number (none) -> XL-1608UBC-04; cost (none) -> 0.004
- D31: value 3.3VA_ON -> LED; Generic Allowed? (none) -> yes; LCSC# (none) -> C965807; Manufacturer (none) -> XINGLIGHT; Part number (none) -> XL-1608UBC-04; cost (none) -> 0.004
- D32: LCSC# (none) -> C12765; Manufacturer onsemi -> LRC; Part number BAT54SLT1G -> LBAT54SLT1G; cost (none) -> 0.01
- D33: value LED_0 -> LED; Generic Allowed? (none) -> yes; LCSC# (none) -> C965807; Manufacturer (none) -> XINGLIGHT; Part number (none) -> XL-1608UBC-04; cost (none) -> 0.004
- D51: value LED_1 -> LED; Generic Allowed? (none) -> yes; LCSC# (none) -> C965807; Manufacturer (none) -> XINGLIGHT; Part number (none) -> XL-1608UBC-04; cost (none) -> 0.004
- J3, NT10, NT11, NT12, TP6, TP7: now not fitted
- R135, R141, R142, R143, R81, R86: Generic Allowed? (none) -> yes; LCSC# (none) -> C60490; Manufacturer (none) -> YAGEO; Part number (none) -> RC0402FR-0710KL; cost (none) -> 0.0007
- R136, R144, R145, R32, R78, R85: Generic Allowed? (none) -> yes, 1% or better; LCSC# (none) -> C106235; Manufacturer (none) -> YAGEO; Part number (none) -> RC0402FR-071KL; cost (none) -> 0.0007
- R137, R99: Generic Allowed? (none) -> yes; LCSC# (none) -> C106231; Manufacturer (none) -> YAGEO; Part number (none) -> RC0402FR-070RL; cost (none) -> 0.0007
- R79, R80: Generic Allowed? (none) -> yes, 1% or better; LCSC# (none) -> C132157; Manufacturer (none) -> YAGEO; Part number (none) -> RC0402FR-0712K1L; cost (none) -> 0.0007
- R82, R83, R84: Generic Allowed? (none) -> yes, 1%, 200v; LCSC# (none) -> C137235; Manufacturer (none) -> YAGEO; Part number (none) -> RC1206FR-07750KL; cost (none) -> 0.004
- U1: Manufacturer (none) -> STM; Part number (none) -> STM32G473QET6; cost (none) -> 7.51
- X1: value SG-8002CE -> 16Mhz; LCSC# (none) -> C390318; Manufacturer (none) -> EPSON; Part number (none) -> SG-8002CE 16.000000MHz PHM; cost (none) -> 1.41
Connections:
- net +3.3V: now also C41.2, U21.5 (OUT)
- net +3.3VA: now also R151.2
- net GND1: now also C24.1, C39.1, C41.1, U21.2 (GND), U6.2 (GND)
- new net: C39.2, R151.1, U6.5 (OUT)
- new net +5VP: C24.2, U21.1 (IN), U21.3 (EN), U6.1 (IN), U6.3 (EN)
Other:
- moved on the sheet: C110, D12, D31, R32, R78

Commit message: update BOM and change transceivers
Parts:
- U1: footprint footprints:QFP40P1600X1600X160-128N -> STM32G473QET6:QFP40P1600X1600X160-128N
- U21, U6: Generic Allowed? (none) -> yes
- X1: Generic Allowed? (none) -> no
Changed lines of the file:
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@@
 			)
 		)
-		(property "Description" "50v"
+		(property "Description" "Unpolarized capacitor"
 			(at 417.83 334.01 0)
 			(effects
@@
 			)
 		)
-		(property "Description" "50v"
+		(property "Description" "Unpolarized capacitor"
 			(at 455.93 334.01 0)
 			(effects
@@
 			)
 		)
-		(property "Description" "50v"
+		(property "Description" "Unpolarized capacitor"
 			(at 355.6 373.38 0)
 			(effects
@@
 			)
 		)
+		(property "Generic Allowed?" "yes"
+			(at 449.58 100.33 0)
+			(effects
+				(font
+					(size 1.27 1.27)
+				)
+				(hide yes)
+			)
+		)
 		(pin "1"
 		)
@@
 			)
 		)
-		(property "Description" "50v"
+		(property "Description" "Unpolarized capacitor"
 			(at 191.77 86.36 0)
 			(effects
@@
 			)
 		)
-		(property "Description" "50v"
+		(property "Description" "Unpolarized capacitor"
 			(at 405.13 334.01 0)
 			(effects
@@
 			)
 		)
-		(property "Description" "50v"
+		(property "Description" "Unpolarized capacitor"
 			(at 191.77 52.07 0)
 			(effects
@@
 			)
 		)
-		(property "Description" "25v"
+		(property "Description" "Unpolarized capacitor"
 			(at 421.64 71.12 0)
 			(effects
@@
 			)
 		)
-		(property "Description" "50v"
+		(property "Description" "Unpolarized capacitor"
 			(at 58.42 142.24 0)
 			(effects
@@
 			)
 		)
-		(property "Footprint" "footprints:QFP40P1600X1600X160-128N"
+		(property "Footprint" "STM32G473QET6:QFP40P1600X1600X160-128N"
 			(at 100.33 273.05 0)
 			(effects
@@
 			)
 		)
-		(property "Description" "50v"
+		(property "Description" "Unpolarized capacitor"
 			(at 157.48 217.17 0)
 			(effects
@@
 			)
 		)
-		(property "Description" "50v"
+		(property "Description" "Unpolarized capacitor"
 			(at 161.29 177.8 0)
 			(effects
@@
 			)
 		)
-		(property "Description" "200v"
+		(property "Description" "Resistor, US symbol"
 			(at 537.21 227.33 0)
 			(effects
@@
 			)
 		)
-		(property "Description" "10v"
+		(property "Description" "Unpolarized capacitor"
 			(at 370.84 373.38 0)
 			(effects
@@
 			)
 		)
-		(property "Footprint" "footprints:QFP40P1600X1600X160-128N"
+		(property "Footprint" "STM32G473QET6:QFP40P1600X1600X160-128N"
 			(at 99.06 326.39 0)
 			(effects
@@
 			)
 		)
-		(property "Description" "50v"
+		(property "Description" "Unpolarized capacitor"
 			(at 379.73 334.01 0)
 			(effects
@@
 			)
 		)
-		(property "Footprint" "footprints:QFP40P1600X1600X160-128N"
+		(property "Footprint" "STM32G473QET6:QFP40P1600X1600X160-128N"
 			(at 100.33 48.26 0)
 			(effects
@@
 			)
 		)
-		(property "Description" "25v"
+		(property "Description" "Unpolarized capacitor"
 			(at 354.33 334.01 0)
 			(effects
@@
 			)
 		)
-		(property "Description" "50v"
+		(property "Description" "Unpolarized capacitor"
 			(at 502.92 260.35 0)
 			(effects
@@
 			)
 		)
-		(property "Footprint" "footprints:QFP40P1600X1600X160-128N"
+		(property "Footprint" "STM32G473QET6:QFP40P1600X1600X160-128N"
 			(at 100.33 217.17 0)
 			(effects
@@
 			)
 		)
-		(property "Footprint" "footprints:QFP40P1600X1600X160-128N"
+		(property "Footprint" "STM32G473QET6:QFP40P1600X1600X160-128N"
 			(at 101.6 106.68 0)
 			(effects
@@
 			)
 		)
+		(property "Generic Allowed?" "yes"
+			(at 449.58 60.96 0)
+			(effects
+				(font
+					(size 1.27 1.27)
+				)
+				(hide yes)
+			)
+		)
 		(pin "1"
 		)
@@
 			)
 		)
-		(property "Description" "25v"
+		(property "Description" "Unpolarized capacitor"
 			(at 466.09 62.23 0)
 			(effects
@@
 			)
 		)
-		(property "Description" "50v"
+		(property "Description" "Unpolarized capacitor"
 			(at 367.03 334.01 0)
 			(effects
@@
 			)
 		)
-		(property "Description" "50v"
+		(property "Description" "Unpolarized capacitor"
 			(at 50.8 157.48 0)
 			(effects
@@
 			)
 		)
-		(property "Footprint" "footprints:QFP40P1600X1600X160-128N"
+		(property "Footprint" "STM32G473QET6:QFP40P1600X1600X160-128N"
 			(at 100.33 374.65 0)
 			(effects
@@
 			)
 		)
-		(property "Description" "200v"
+		(property "Description" "Resistor, US symbol"
 			(at 537.21 242.57 0)
 			(effects
@@
 			)
 		)
-		(property "Description" "50v"
+		(property "Description" "Unpolarized capacitor"
 			(at 383.54 373.38 0)
 			(effects
@@
 			)
 		)
-		(property "Description" "10v"
+		(property "Description" "Unpolarized capacitor"
 			(at 342.9 373.38 0)
 			(effects
@@
 			)
 		)
-		(property "Footprint" "footprints:QFP40P1600X1600X160-128N"
+		(property "Footprint" "STM32G473QET6:QFP40P1600X1600X160-128N"
 			(at 99.06 163.83 0)
 			(effects
@@
 			)
 		)
-		(property "Description" "50v"
+		(property "Description" "Unpolarized capacitor"
 			(at 191.77 120.65 0)
 			(effects
@@
 			)
 		)
-		(property "Description" "50v"
+		(property "Description" "Unpolarized capacitor"
 			(at 351.79 68.58 0)
 			(effects
@@
 			)
 		)
+		(property "Generic Allowed?" "no"
+			(at 152.4 190.5 0)
+			(effects
+				(font
+					(size 1.27 1.27)
+				)
+				(hide yes)
+			)
+		)
 		(pin "1"
 		)
@@
 			)
 		)
-		(property "Description" "200v"
+		(property "Description" "Resistor, US symbol"
 			(at 537.21 234.95 0)
 			(effects
@@
 			)
 		)
-		(property "Description" "50v"
+		(property "Description" "Unpolarized capacitor"
 			(at 392.43 334.01 0)
 			(effects
@@
 			)
 		)
-		(property "Description" "50v"
+		(property "Description" "Unpolarized capacitor"
 			(at 430.53 334.01 0)
 			(effects
@@
 			)
 		)
-		(property "Description" "50v"
+		(property "Description" "Unpolarized capacitor"
 			(at 443.23 334.01 0)
 			(effects
@@
 			)
 		)
-		(property "Footprint" "footprints:QFP40P1600X1600X160-128N"
+		(property "Footprint" "STM32G473QET6:QFP40P1600X1600X160-128N"
 			(at 311.15 336.55 0)
 			(effects
@@
 			)
 		)
-		(property "Description" "50v"
+		(property "Description" "Unpolarized capacitor"
 			(at 83.82 391.16 0)
 			(effects
@@
 			)
 		)
-		(property "Description" "25v"
+		(property "Description" "Unpolarized capacitor"
 			(at 466.09 101.6 0)
 			(effects
@@
 			)
 		)
-		(property "Description" "50v"
+		(property "Description" "Unpolarized capacitor"
 			(at 166.37 194.31 0)
 			(effects
@@
 			)
 		)
-		(property "Description" "25v"
+		(property "Description" "Unpolarized capacitor"
 			(at 497.84 104.14 0)
 			(effects
