File: KiCad/high voltage servo drive 3ch/microcontroller.kicad_sch (KiCad schematic)
At the start: 63 parts, among them J3 Conn_ARM_SWD_TagConnect_TC2030, U1 STM32G473QET6, U21 TLV75733PDBV, U6 TLV75733PDBV, X1 25Mhz

Commit message: update bom
Parts:
- U1: value STM32G473QET6 -> STM32G474QET6; LCSC# (none) -> C730129; Part number STM32G473QET6 -> STM32G474QET6; cost 7.51 -> 9.836
Changed lines of the file:
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@@
 			)
 		)
-		(property "Value" "STM32G473QET6"
+		(property "Value" "STM32G474QET6"
 			(at 109.22 275.5899 0)
 			(effects
@@
 			)
 		)
-		(property "cost" "7.51"
+		(property "cost" "9.836"
 			(at 100.33 273.05 0)
 			(effects
@@
 			)
 		)
-		(property "Part number" "STM32G473QET6"
+		(property "Part number" "STM32G474QET6"
 			(at 100.33 273.05 0)
 			(effects
@@
 			)
 		)
+		(property "LCSC#" "C730129"
+			(at 100.33 273.05 0)
+			(effects
+				(font
+					(size 1.27 1.27)
+				)
+				(hide yes)
+			)
+		)
 		(pin "82"
 		)
@@
 			)
 		)
-		(property "Value" "STM32G473QET6"
+		(property "Value" "STM32G474QET6"
 			(at 110.49 328.9299 0)
 			(effects
@@
 			)
 		)
-		(property "cost" "7.51"
+		(property "cost" "9.836"
 			(at 99.06 326.39 0)
 			(effects
@@
 			)
 		)
-		(property "Part number" "STM32G473QET6"
+		(property "Part number" "STM32G474QET6"
 			(at 99.06 326.39 0)
 			(effects
@@
 			)
 		)
+		(property "LCSC#" "C730129"
+			(at 99.06 326.39 0)
+			(effects
+				(font
+					(size 1.27 1.27)
+				)
+				(hide yes)
+			)
+		)
 		(pin "82"
 		)
@@
 			)
 		)
-		(property "Value" "STM32G473QET6"
+		(property "Value" "STM32G474QET6"
 			(at 109.22 50.7999 0)
 			(effects
@@
 			)
 		)
-		(property "cost" "7.51"
+		(property "cost" "9.836"
 			(at 100.33 48.26 0)
 			(effects
@@
 			)
 		)
-		(property "Part number" "STM32G473QET6"
+		(property "Part number" "STM32G474QET6"
 			(at 100.33 48.26 0)
 			(effects
@@
 			)
 		)
+		(property "LCSC#" "C730129"
+			(at 100.33 48.26 0)
+			(effects
+				(font
+					(size 1.27 1.27)
+				)
+				(hide yes)
+			)
+		)
 		(pin "82"
 		)
@@
 			)
 		)
-		(property "Value" "STM32G473QET6"
+		(property "Value" "STM32G474QET6"
 			(at 109.22 219.7099 0)
 			(effects
@@
 			)
 		)
-		(property "cost" "7.51"
+		(property "cost" "9.836"
 			(at 100.33 217.17 0)
 			(effects
@@
 			)
 		)
-		(property "Part number" "STM32G473QET6"
+		(property "Part number" "STM32G474QET6"
 			(at 100.33 217.17 0)
 			(effects
@@
 			)
 		)
+		(property "LCSC#" "C730129"
+			(at 100.33 217.17 0)
+			(effects
+				(font
+					(size 1.27 1.27)
+				)
+				(hide yes)
+			)
+		)
 		(pin "82"
 		)
@@
 			)
 		)
-		(property "Value" "STM32G473QET6"
+		(property "Value" "STM32G474QET6"
 			(at 110.49 109.2199 0)
 			(effects
@@
 			)
 		)
-		(property "cost" "7.51"
+		(property "cost" "9.836"
 			(at 101.6 106.68 0)
 			(effects
@@
 			)
 		)
-		(property "Part number" "STM32G473QET6"
+		(property "Part number" "STM32G474QET6"
 			(at 101.6 106.68 0)
 			(effects
@@
 			)
 		)
+		(property "LCSC#" "C730129"
+			(at 101.6 106.68 0)
+			(effects
+				(font
+					(size 1.27 1.27)
+				)
+				(hide yes)
+			)
+		)
 		(pin "82"
 		)
@@
 			)
 		)
-		(property "Value" "STM32G473QET6"
+		(property "Value" "STM32G474QET6"
 			(at 109.22 375.9199 0)
 			(effects
@@
 			)
 		)
-		(property "cost" "7.51"
+		(property "cost" "9.836"
 			(at 100.33 374.65 0)
 			(effects
@@
 			)
 		)
-		(property "Part number" "STM32G473QET6"
+		(property "Part number" "STM32G474QET6"
 			(at 100.33 374.65 0)
 			(effects
@@
 			)
 		)
+		(property "LCSC#" "C730129"
+			(at 100.33 374.65 0)
+			(effects
+				(font
+					(size 1.27 1.27)
+				)
+				(hide yes)
+			)
+		)
 		(pin "82"
 		)
@@
 			)
 		)
-		(property "Value" "STM32G473QET6"
+		(property "Value" "STM32G474QET6"
 			(at 113.03 166.3699 0)
 			(effects
@@
 			)
 		)
-		(property "cost" "7.51"
+		(property "cost" "9.836"
 			(at 99.06 163.83 0)
 			(effects
@@
 			)
 		)
-		(property "Part number" "STM32G473QET6"
+		(property "Part number" "STM32G474QET6"
 			(at 99.06 163.83 0)
 			(effects
@@
 			)
 		)
+		(property "LCSC#" "C730129"
+			(at 99.06 163.83 0)
+			(effects
+				(font
+					(size 1.27 1.27)
+				)
+				(hide yes)
+			)
+		)
 		(pin "82"
 		)
@@
 			)
 		)
-		(property "Value" "STM32G473QET6"
+		(property "Value" "STM32G474QET6"
 			(at 311.15 323.85 0)
 			(effects
@@
 			)
 		)
-		(property "cost" "7.51"
+		(property "cost" "9.836"
 			(at 311.15 336.55 0)
 			(effects
@@
 			)
 		)
-		(property "Part number" "STM32G473QET6"
+		(property "Part number" "STM32G474QET6"
 			(at 311.15 336.55 0)
 			(effects
@@
 			(at 311.15 336.55 0)
 			(effects
+				(font
+					(size 1.27 1.27)
+				)
+				(hide yes)
+			)
+		)
+		(property "LCSC#" "C730129"
+			(at 311.15 336.55 0)
+			(effects
