File: KiCad/high voltage servo drive 3ch/power_connectors.kicad_sch (KiCad schematic)
At the start: 13 parts, among them J4 MOTOR_A, J5 MOTOR_B, J6 MOTOR_C, J7 DC BUS

Commit message: prepare rev0.1 for manufacturing
Parts:
- added C204, C206: 22uf, Capacitor_SMD:C_1206_3216Metric, symbol Device:C
- added C205: .1uf, Capacitor_SMD:C_0402_1005Metric, symbol Device:C
- added C207: .1uf, Capacitor_SMD:C_1812_4532Metric, symbol Device:C
- added D11: LED, LED_SMD:LED_0603_1608Metric, symbol Device:LED
- added D52, D53: ES1J, Diode_SMD:D_SMA, symbol Device:D
- added L9: L, Inductor_THT:L_Radial_D7.2mm_P3.00mm_Murata_1700, symbol Device:L
- added R150, R31: 10k, Resistor_SMD:R_0402_1005Metric, symbol Device:R_US
- added R152: 1k, Resistor_SMD:R_0402_1005Metric, symbol Device:R_US
- added TP1: GATE_SUPPLY, TestPoint:TestPoint_Pad_D2.0mm, symbol Connector:TestPoint
- added U20: LNK306D, Package_SO:PowerIntegrations_SO-8C, symbol Regulator_Switching:LNK306D
- C130: footprint Capacitor_THT:C_Rect_L18.0mm_W11.0mm_P15.00mm_FKS3_FKP3 -> Capacitor_THT:C_Rect_L26.5mm_W10.5mm_P22.50mm_MKS4; Generic Allowed? (none) -> yes; LCSC# C19190310 -> C2928857; Manufacturer (none) -> KYET; Part number (none) -> MPB105J2J2201; cost (none) -> 0.23; now not fitted
- C131, C132, C133, C134, C135, C21: Generic Allowed? (none) -> no
- J4, J5, J6: Generic Allowed? (none) -> no; LCSC# (none) -> C7422679; Manufacturer (none) -> DORABO; Part number (none) -> DB3ERC-7.62-3P-GN; cost (none) -> 0.79
- J7: Generic Allowed? (none) -> no; Manufacturer (none) -> DORABO; Part number (none) -> DB3ERC-7.62-2P-GN; cost (none) -> 0.56
- L7, L8: Generic Allowed? (none) -> yes; Manufacturer (none) -> COILMX; Part number (none) -> MS1050-R22M; cost (none) -> 0.14
Connections:
- net GND1: now also C206.1, C207.2, D11.1 (K), D52.2 (A)
- net VBUS: now also C207.1, U20.4 (D)
- new net: C204.1, C205.1, D52.1 (K), L9.1, R152.1, U20.5 (S), U20.6 (S), U20.7 (S), U20.8 (S)
- new net: R150.1, R152.2, U20.2 (FB)
- new net: C204.2, D53.1 (K), R150.2
- new net: D11.2 (A), R31.1
- new net: C205.2, U20.1 (BP)
- new net +GATE_SUPPLY: C206.2, D53.2 (A), L9.2, R31.2, TP1.1
Other:
- note added: "1.65v FBK target voltage 11k: 18.15v 9.2k: 15.18v"
- note added: "GATE_SUPPLY voltage must be set according to which IPMs are used IGBT: 15v SiC: 18v"

Commit message: fix DRC issues
Parts:
- C131, C132, C133, C134, C135, C21: footprint footprints:C_Rect_L32mm_W18.0mm_P27.50mm_MKS4 -> footprints:C_Rect_L32mm_W16.0mm_P27.50mm
Changed lines of the file:
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@@
 			)
 		)
-		(property "Footprint" "footprints:C_Rect_L32mm_W18.0mm_P27.50mm_MKS4"
+		(property "Footprint" "footprints:C_Rect_L32mm_W16.0mm_P27.50mm"
 			(at 150.8252 46.99 0)
 			(effects
@@
 			)
 		)
-		(property "Footprint" "footprints:C_Rect_L32mm_W18.0mm_P27.50mm_MKS4"
+		(property "Footprint" "footprints:C_Rect_L32mm_W16.0mm_P27.50mm"
 			(at 139.3952 46.99 0)
 			(effects
@@
 			)
 		)
-		(property "Footprint" "footprints:C_Rect_L32mm_W18.0mm_P27.50mm_MKS4"
+		(property "Footprint" "footprints:C_Rect_L32mm_W16.0mm_P27.50mm"
 			(at 116.5352 46.99 0)
 			(effects
@@
 			)
 		)
-		(property "Footprint" "footprints:C_Rect_L32mm_W18.0mm_P27.50mm_MKS4"
+		(property "Footprint" "footprints:C_Rect_L32mm_W16.0mm_P27.50mm"
 			(at 93.6752 46.99 0)
 			(effects
@@
 			)
 		)
-		(property "Footprint" "footprints:C_Rect_L32mm_W18.0mm_P27.50mm_MKS4"
+		(property "Footprint" "footprints:C_Rect_L32mm_W16.0mm_P27.50mm"
 			(at 105.1052 46.99 0)
 			(effects
@@
 			)
 		)
-		(property "Footprint" "footprints:C_Rect_L32mm_W18.0mm_P27.50mm_MKS4"
+		(property "Footprint" "footprints:C_Rect_L32mm_W16.0mm_P27.50mm"
 			(at 127.9652 46.99 0)
 			(effects

Commit message: update BOM and change transceivers
Parts:
- C130: now fitted
- U20: footprint Package_SO:PowerIntegrations_SO-8C -> Package_SO:PowerIntegrations_SO-8B; Generic Allowed? (none) -> no
Changed lines of the file:
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@@
 			)
 		)
-		(property "Description" "25v"
+		(property "Description" "Unpolarized capacitor"
 			(at 193.04 148.59 0)
 			(effects
@@
 			)
 		)
-		(property "Description" "1kv"
+		(property "Description" "Unpolarized capacitor"
 			(at 77.47 146.05 0)
 			(effects
@@
 		(in_bom yes)
 		(on_board yes)
-		(dnp yes)
+		(dnp no)
 		(fields_autoplaced yes)
 		(property "Reference" "C130"
@@
 			)
 		)
-		(property "Footprint" "Package_SO:PowerIntegrations_SO-8C"
+		(property "Footprint" "Package_SO:PowerIntegrations_SO-8B"
 			(at 106.68 142.24 0)
 			(effects
@@
 		)
 		(property "cost" "0.62"
+			(at 106.68 142.24 0)
+			(effects
+				(font
+					(size 1.27 1.27)
+				)
+				(hide yes)
+			)
+		)
+		(property "Generic Allowed?" "no"
 			(at 106.68 142.24 0)
 			(effects
@@
 			)
 		)
-		(property "Description" "25v"
+		(property "Description" "Unpolarized capacitor"
 			(at 157.48 134.62 0)
 			(effects
@@
 			)
 		)
-		(property "Description" "50v"
+		(property "Description" "Unpolarized capacitor"
 			(at 121.92 135.89 0)
 			(effects
