File: KiCad/high voltage servo drive 3ch/power_connectors.kicad_sch (KiCad schematic)
At the start: 26 parts, among them J4 MOTOR_A, J5 MOTOR_B, J6 MOTOR_C, J7 DC BUS, U20 LNK306D

Commit message: update bom
Parts:
- C131, C132, C133, C134, C135, C21: Manufacturer (none) -> XIAMEN FARATRONIC; Part number (none) -> D3D1U106KB00C00; cost (none) -> 1.124; now not fitted
Changed lines of the file:
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@@
 		(in_bom yes)
 		(on_board yes)
-		(dnp no)
+		(dnp yes)
 		(fields_autoplaced yes)
 		(property "Reference" "C135"
@@
 			)
 		)
-		(property "cost" ""
+		(property "cost" "1.124"
 			(at 149.86 43.18 0)
 			(effects
@@
 		)
 		(property "Generic Allowed?" "no"
+			(at 149.86 43.18 0)
+			(effects
+				(font
+					(size 1.27 1.27)
+				)
+				(hide yes)
+			)
+		)
+		(property "Manufacturer" "XIAMEN FARATRONIC"
+			(at 149.86 43.18 0)
+			(effects
+				(font
+					(size 1.27 1.27)
+				)
+				(hide yes)
+			)
+		)
+		(property "Part number" "D3D1U106KB00C00"
 			(at 149.86 43.18 0)
 			(effects
@@
 		(in_bom yes)
 		(on_board yes)
-		(dnp no)
+		(dnp yes)
 		(fields_autoplaced yes)
 		(property "Reference" "C134"
@@
 			)
 		)
-		(property "cost" ""
+		(property "cost" "1.124"
 			(at 138.43 43.18 0)
 			(effects
@@
 		)
 		(property "Generic Allowed?" "no"
+			(at 138.43 43.18 0)
+			(effects
+				(font
+					(size 1.27 1.27)
+				)
+				(hide yes)
+			)
+		)
+		(property "Manufacturer" "XIAMEN FARATRONIC"
+			(at 138.43 43.18 0)
+			(effects
+				(font
+					(size 1.27 1.27)
+				)
+				(hide yes)
+			)
+		)
+		(property "Part number" "D3D1U106KB00C00"
 			(at 138.43 43.18 0)
 			(effects
@@
 		(in_bom yes)
 		(on_board yes)
-		(dnp no)
+		(dnp yes)
 		(fields_autoplaced yes)
 		(property "Reference" "C132"
@@
 			)
 		)
-		(property "cost" ""
+		(property "cost" "1.124"
 			(at 115.57 43.18 0)
 			(effects
@@
 		)
 		(property "Generic Allowed?" "no"
+			(at 115.57 43.18 0)
+			(effects
+				(font
+					(size 1.27 1.27)
+				)
+				(hide yes)
+			)
+		)
+		(property "Manufacturer" "XIAMEN FARATRONIC"
+			(at 115.57 43.18 0)
+			(effects
+				(font
+					(size 1.27 1.27)
+				)
+				(hide yes)
+			)
+		)
+		(property "Part number" "D3D1U106KB00C00"
 			(at 115.57 43.18 0)
 			(effects
@@
 		(in_bom yes)
 		(on_board yes)
-		(dnp no)
+		(dnp yes)
 		(fields_autoplaced yes)
 		(property "Reference" "C21"
@@
 			)
 		)
-		(property "cost" ""
+		(property "cost" "1.124"
 			(at 92.71 43.18 0)
 			(effects
@@
 		)
 		(property "Generic Allowed?" "no"
+			(at 92.71 43.18 0)
+			(effects
+				(font
+					(size 1.27 1.27)
+				)
+				(hide yes)
+			)
+		)
+		(property "Manufacturer" "XIAMEN FARATRONIC"
+			(at 92.71 43.18 0)
+			(effects
+				(font
+					(size 1.27 1.27)
+				)
+				(hide yes)
+			)
+		)
+		(property "Part number" "D3D1U106KB00C00"
 			(at 92.71 43.18 0)
 			(effects
@@
 		(in_bom yes)
 		(on_board yes)
-		(dnp no)
+		(dnp yes)
 		(fields_autoplaced yes)
 		(property "Reference" "C131"
@@
 			)
 		)
-		(property "cost" ""
+		(property "cost" "1.124"
 			(at 104.14 43.18 0)
 			(effects
@@
 		)
 		(property "Generic Allowed?" "no"
+			(at 104.14 43.18 0)
+			(effects
+				(font
+					(size 1.27 1.27)
+				)
+				(hide yes)
+			)
+		)
+		(property "Manufacturer" "XIAMEN FARATRONIC"
+			(at 104.14 43.18 0)
+			(effects
+				(font
+					(size 1.27 1.27)
+				)
+				(hide yes)
+			)
+		)
+		(property "Part number" "D3D1U106KB00C00"
 			(at 104.14 43.18 0)
 			(effects
@@
 		(in_bom yes)
 		(on_board yes)
-		(dnp no)
+		(dnp yes)
 		(fields_autoplaced yes)
 		(property "Reference" "C133"
@@
 			)
 		)
-		(property "cost" ""
+		(property "cost" "1.124"
 			(at 127 43.18 0)
 			(effects
@@
 			(at 127 43.18 0)
 			(effects
+				(font
+					(size 1.27 1.27)
+				)
+				(hide yes)
+			)
+		)
+		(property "Manufacturer" "XIAMEN FARATRONIC"
+			(at 127 43.18 0)
+			(effects
+				(font
+					(size 1.27 1.27)
+				)
+				(hide yes)
+			)
+		)
+		(property "Part number" "D3D1U106KB00C00"
+			(at 127 43.18 0)
+			(effects
