File: KiCad/high voltage servo drive 3ch/inverter_A.kicad_sch (KiCad schematic)
At the start: 50 parts, among them U2 IPM

Commit message: add rev 0.2 changes and rev 0.1 mfg files
Parts:
- removed R138: 5.1k, Resistor_SMD:R_0402_1005Metric, symbol Device:R_US
- added R25: 12.1k, Resistor_SMD:R_0402_1005Metric, symbol Device:R_US
- R7: value 5.1k -> 12.1k; Generic Allowed? yes -> yes, 1% or better; LCSC# C105873 -> C132157; Part number RC0402JR-075K1L -> RC0402FR-0712K1L; cost 0.0006 -> 0.0007
- U2: footprint DIP39_54.5X31.0_MODGC_OSI -> footprints:DIP39_54.5X31.0_MODGC_OSI; Generic Allowed? (none) -> no; now not fitted
Connections:
- net GND1: now also R7.2; no longer R7.1
- net TEMP: now also R7.1, R25.1
- net at C17.1, U2.20 (VTS): now also R25.2; no longer R7.2
Other:
- moved on the sheet: C195
